File: KICAD Projects/General/Primis_Turrim/TurrimX3/TurrimX3.kicad_sch (KiCad schematic)
At the start: 37 parts, among them IC1 LSM6DSV16XTR, IC2 QMC6309, J3 Conn_01x05_Pin, J4 USB_C_Receptacle_USB2.0_16P, U1 nRF52833_QDxx, U2 TLV70036_SOT23-5, Y2 Crystal_GND24

Commit message: Big Update
-Added Versipellis pictures
-Split Turrim into 2 versions, a simple, cheap 1 port version and a more complex 4 port hub version.
-Started work on Locus
Parts:
- removed C10, C12, C13: 100nF, Capacitor_SMD:C_0603_1608Metric, symbol Device:C
- removed C11, C29: 1.0uF, Capacitor_SMD:C_0805_2012Metric, symbol Device:C
- removed C15, C19: 1uF, Capacitor_SMD:C_0603_1608Metric, symbol Device:C
- removed C16, C18: 4.7K, Capacitor_SMD:C_0603_1608Metric, symbol Device:C
- removed C17: 2.2uF, Capacitor_SMD:C_0603_1608Metric, symbol Device:C
- removed C30: N.C., Capacitor_SMD:C_0603_1608Metric, symbol Device:C
- removed C31: 100pF, Capacitor_SMD:C_0805_2012Metric, symbol Device:C
- removed D1: WS2812B, LED_SMD:LED_WS2812B_PLCC4_5.0x5.0mm_P3.2mm, symbol LED:WS2812B
- removed H1, H2, H3, H4: MountingHole, MountingHole:MountingHole_2.2mm_M2, symbol Mechanical:MountingHole
- removed IC1: LSM6DSV16XTR, LSM6DSV16BXTR, symbol LSM6DSV16XTR:LSM6DSV16XTR
- removed IC2: QMC6309, QMC6309, symbol QMC6309:QMC6309
- removed J3: Conn_01x05_Pin, Connector_PinHeader_1.00mm:PinHeader_1x05_P1.00mm_Vertical, symbol Connector:Conn_01x05_Pin
- removed J4: USB_C_Receptacle_USB2.0_16P, symbol Connector:USB_C_Receptacle_USB2.0_16P
- removed L1: 4.7nH, Inductor_SMD:L_0603_1608Metric, symbol Device:L
- removed L2: 2.2nH, Inductor_SMD:L_0603_1608Metric, symbol Device:L
- removed R8: 2R2, Resistor_SMD:R_0805_2012Metric, symbol Device:R
- removed R9: 10k, Resistor_SMD:R_0805_2012Metric, symbol Device:R
- removed U1: nRF52833_QDxx, Package_DFN_QFN:QFN-40-1EP_5x5mm_P0.4mm_EP3.6x3.6mm, symbol MCU_Nordic:nRF52833_QDxx
- removed U2: TLV70036_SOT23-5, Package_TO_SOT_SMD:SOT-23-5, symbol Regulator_Linear:TLV70036_SOT23-5
- removed Y2: Crystal_GND24, symbol Device:Crystal_GND24
- added D1, D2, D3, D4: LED, LED_SMD:LED_0603_1608Metric, symbol Device:LED
- added F1: Polyfuse, Fuse:Fuse_1206_3216Metric, symbol Device:Polyfuse
- added J1: USB_C_Receptacle_USB2.0_16P, Connector_USB:USB_C_Receptacle_HRO_TYPE-C-31-M-12, symbol Connector:USB_C_Receptacle_USB2.0_16P
- added J2, J3, J4, J5: USB_A, Connector_USB:USB_A_Molex_105057_Vertical, symbol Connector:USB_A
- added R1, R2: 5.1K, Resistor_SMD:R_0805_2012Metric, symbol Device:R
- added R3, R4, R5, R6: 4.7k, Resistor_SMD:R_0805_2012Metric, symbol Device:R
- added U1: CH334F, Package_DFN_QFN:QFN-24-1EP_4x4mm_P0.5mm_EP2.7x2.7mm, symbol Interface_USB:CH334F
- added Y1: 12MHZ, Crystal:Crystal_SMD_2016-4Pin_2.0x1.6mm, symbol Device:Crystal
- C1: value 100nF -> 10uF; footprint Capacitor_SMD:C_0603_1608Metric -> Capacitor_SMD:C_0805_2012Metric
- C2: value 4.7uF -> 1uF; footprint Capacitor_SMD:C_0805_2012Metric -> Capacitor_SMD:C_0603_1608Metric
- C3: value 12pF -> 10uF
- C4: value 12pF -> 0.1uF; footprint Capacitor_SMD:C_0805_2012Metric -> Capacitor_SMD:C_0603_1608Metric
- C5: value 0.8pF -> 220uF; footprint Capacitor_SMD:C_0603_1608Metric -> Capacitor_SMD:C_0805_2012Metric
- C6: value 1.0pF -> 100uF; footprint Capacitor_SMD:C_0603_1608Metric -> Capacitor_SMD:C_0805_2012Metric
- C7, C9: value 4.7uF -> 100uF
- C8: value 100nF -> 100uF; footprint Capacitor_SMD:C_0603_1608Metric -> Capacitor_SMD:C_0805_2012Metric
Connections:
- net D+: now also J1.A6 (D+), J1.B6 (D+), U1.15 (DPU+)
- net D-: now also J1.A7 (D-), J1.B7 (D-), U1.14 (DMU-)
- net GND: now also C1.2, C3.2, C4.2, C6.2, C8.2, J1.A1 (GND), J1.A12 (GND), J1.B1 (GND), J1.B12 (GND), J1.SH (SHIELD), J2.4 (GND), J2.SH (Shield), J3.4 (GND), J3.SH (Shield), J4.4 (GND), J4.SH (Shield), J5.4 (GND), J5.SH (Shield), R1.2, R2.2, U1.25 (GND); no longer C1.1, C3.1, C4.1, C6.1, C8.1
- net VBUS: now also C5.2, C6.1, C7.1, C8.1, C9.1, D1.2 (A), D2.2 (A), D3.2 (A), D4.2 (A), F1.2, J2.1 (VBUS), J3.1 (VBUS), J4.1 (VBUS), J5.1 (VBUS)
- net +3.3V: now reaches C2.1
- net +3.3V: now also C3.1, U1.20 (VDD33_{LDO})
- removed net VDD_nRF: C8.2, C9.1
- new net: D4.1 (K), R6.1
- new net: R6.2, U1.21 (LED4/SDA)
- new net: D3.1 (K), R5.1
- new net: R5.2, U1.13 (LED3/SCL)
- new net: R3.2, U1.22 (LED1)
- new net: R4.2, U1.23 (LED2)
- new net: U1.3 (XO), Y1.2
- new net: U1.4 (XI), Y1.1
- new net: J1.B5 (CC2), R2.1
- new net: D1.1 (K), R3.1
- new net: D2.1 (K), R4.1
- new net: J1.A5 (CC1), R1.1
- new net +5V: C1.1, C4.1, F1.1, J1.A4 (VBUS), J1.A9 (VBUS), J1.B4 (VBUS), J1.B9 (VBUS), U1.19 (V5)
- new net DDOWN+: J2.3 (D+), U1.12 (DP1+)
- new net DDOWN-: J2.2 (D-), U1.11 (DM1-)
- new net DDOWN2+: J4.3 (D+), U1.10 (DP2+)
- new net DDOWN2-: J4.2 (D-), U1.9 (DM2-)
- new net DDOWN3+: J3.3 (D+), U1.8 (DP3+)
- new net DDOWN3-: J3.2 (D-), U1.7 (DM3-)
- new net DDOWN4+: J5.3 (D+), U1.6 (DP4+)
- new net DDOWN4-: J5.2 (D-), U1.5 (DM4-)
- no-connect marks 2 -> 6
Other:
- title: Locus -> Dongle Dock x4
