File: KICAD Projects/General/PI3_Carrier/PI3_Carrier.kicad_sch (KiCad schematic)
At the start: 0 parts

Commit message: CleanUp
-Added Locus EV1 STEP and STL files
-Added Locus PCB picture
-Added very early work on PI3 carrier board
-Added nearly complete VeriMini kicad project
-Added extra details to README
Parts:
- added C1, C2, C3, C4: 100nf, symbol Device:C
- added D1, D2, D3, D4: WS2812B-2020, LED_SMD:LED_WS2812B-2020_PLCC4_2.0x2.0mm, symbol LED:WS2812B-2020
- added X1: AFA07-S15FCA-00, primis2:AFA07-S15FCA-00, symbol primis2:AFA07-S15FCA-00
Connections:
- new net: C4.2, D4.4 (VDD)
- new net: C3.2, D2.4 (VDD)
- new net: C2.2, D3.4 (VDD)
- new net: C1.2, D1.4 (VDD)
- new net CSI_CLKN: X1.8
- new net CSI_CLKP: X1.9
- new net CSI_D0N: X1.2
- new net CSI_D0P: X1.3
- new net CSI_D1N: X1.5
- new net CSI_D1P: X1.6
- new net ENABLE: X1.11
- new net GND: D1.2 (VSS), D2.2 (VSS), D3.2 (VSS), D4.2 (VSS), X1.1, X1.10, X1.16, X1.17, X1.4, X1.7
- new net POWER: C1.1, C2.1, C3.1, C4.1, X1.15
- new net SCL: X1.13
- new net SDA: X1.14
- no-connect marks 0 -> 5
