File: KICAD Projects/Primis_Locus/_restore_backup_2026-10-03T20-47-52-471/Locus.kicad_pcb (KiCad board)
At the start: 4 copper layers, 40 x 40 mm, 65 parts, among them J1 Conn_ARM_SWD_TagConnect_TC203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, J2 S2B-PH-SM4-TB_LF_SN, J4 USB_C_Receptacle_USB2.0_16P, SW1 SW_DPST_x2, U1 nRF52833_QDxx, U2 LSM6DSV16XTR, U3 LP5817DRLR, U5 MCP73831T-2ATI_OT, Y1 32.768kHz, Y2 32MHz

Commit message: ev2 wip1
Parts:
- removed C15: 1u, Capacitor_SMD:C_0402_1005Metric
- added R4: 4.7k, Resistor_SMD:R_0402_1005Metric, F.Cu at (203.0, 49.8)
- moved G*** 33.1 mm to (191.5, 84.2)
- moved TP4 15.6 mm to (208.0, 82.8)
- moved G*** 14.8 mm to (215.0, 63.8)
- moved R2 7.77 mm to (199.5, 49.8)
- moved C13 7.66 mm to (204.5, 53.5), turned to 90 degrees
- moved D5 7.40 mm to (226.2, 83.3), turned to 0 degrees
- moved R1 7.21 mm to (201.2, 49.8), turned to -90 degrees
- moved R13 6.75 mm to (203.2, 61.0)
- moved R10 6.03 mm to (210.8, 81.3), turned to 180 degrees
- moved D2 5.45 mm to (201.3, 58.2), turned to 0 degrees
- moved J1 5.41 mm to (214.5, 78.7), turned to 0 degrees
- moved U2 5.00 mm to (201.2, 53.2), turned to 0 degrees
- moved R15 4.79 mm to (198.5, 57.2), turned to 180 degrees
- moved H3 4.00 mm to (184.5, 84.2)
- moved C10 4.00 mm to (205.0, 59.8)
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Connections:
- D3 pad 2: VDDH -> unconnected-(D3-A-Pad2)
- D4 pad 2: VDDH -> unconnected-(D4-A-Pad2)
- D5 pad 2: VDDH -> unconnected-(D5-A-Pad2)
- R13 pad 2: Net-(U1-AIN7/P0.31) -> Net-(U1-AIN4/P0.28)
- R14 pad 2: Net-(U1-AIN2/P0.04) -> Net-(U1-AIN5/P0.29)
- R15 pad 2: Net-(U1-AIN3/P0.05) -> Net-(U1-AIN6/P0.30)
- U1 pad 14: unconnected-(U1-P0.15-Pad14) -> INT
- U1 pad 31: INT -> unconnected-(U1-AIN1/P0.03-Pad31)
- U1 pad 32: MISO -> unconnected-(U1-AIN0/P0.02-Pad32)
- U1 pad 33: MOSI -> Net-(U1-AIN4/P0.28)
- U1 pad 34: SCK -> Net-(U1-AIN5/P0.29)
- U1 pad 35: CS -> Net-(U1-AIN6/P0.30)
- U1 pad 36: Net-(U1-AIN7/P0.31) -> unconnected-(U1-AIN7/P0.31-Pad36)
- U1 pad 4: Net-(U1-AIN2/P0.04) -> unconnected-(U1-AIN2/P0.04-Pad4)
- U1 pad 5: Net-(U1-AIN3/P0.05) -> unconnected-(U1-AIN3/P0.05-Pad5)
- U2 pad 1: MISO -> GND
- U2 pad 13: SCK -> SCL
- U2 pad 14: MOSI -> SDA
- U3 pad 1: SCL -> unconnected-(U3-SCL-Pad1)
- U3 pad 2: SDA -> unconnected-(U3-SDA-Pad2)
Routing:
- net VDDH: track 111.7 -> 35.7 mm, vias 4 -> 2
- net Net-(D3-K): track 33.2 -> 0.00 mm, vias 2 -> 0
- net SDA: track 21.1 -> 40.6 mm
- net INT: track 10.5 -> 29.9 mm, vias 0 -> 2
- net VDD_nRF: track 88.5 -> 107.8 mm
- net SCL: track 21.5 -> 39.7 mm
- net Net-(D5-K): track 33.4 -> 16.2 mm, vias 2 -> 1
- net Net-(U1-AIN3/P0.05): track 10.5 -> 0.00 mm, vias 2 -> 0
- net Net-(U1-AIN6/P0.30): track 0.00 -> 9.64 mm, vias 0 -> 2
- net Net-(U1-AIN2/P0.04): track 9.20 -> 0.00 mm, vias 2 -> 0
- net Net-(U1-AIN7/P0.31): track 8.95 -> 0.00 mm
- net Net-(U1-AIN5/P0.29): track 0.00 -> 8.36 mm, vias 0 -> 2
- net MISO: track 6.19 -> 0.00 mm
- net Net-(U1-P0.18/~{RESET}): track 8.93 -> 15.1 mm
- net SCK: track 6.19 -> 0.00 mm
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