File: KICAD Projects/Primis_Locus/_restore_backup_2026-10-03T20-47-52-471/Locus.kicad_sch (KiCad schematic)
At the start: 61 parts, among them J1 Conn_ARM_SWD_TagConnect_TC203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, J2 S2B-PH-SM4-TB_LF_SN, J4 USB_C_Receptacle_USB2.0_16P, SW1 SW_DPST_x2, U1 nRF52833_QDxx, U2 LSM6DSV16XTR, U3 LP5817DRLR, U5 MCP73831T-2ATI_OT, Y1 32.768kHz, Y2 32MHz

Commit message: ev2 wip1
Parts:
- removed C15: 1u, Capacitor_SMD:C_0402_1005Metric, symbol Device:C
- added R4: 4.7k, Resistor_SMD:R_0402_1005Metric, symbol Device:R
Connections:
- net CS: now also R4.2; no longer U1.35 (AIN6/P0.30)
- net GND: now also U2.1 (SDO/SA0)
- net INT: now also U1.14 (P0.15); no longer U1.31 (AIN1/P0.03)
- net SCL: now also U2.13 (SCL); no longer U3.1 (SCL)
- net SDA: now also U2.14 (SDA); no longer U3.2 (SDA)
- net VDDH: no longer D3.2 (A), D4.2 (A), D5.2 (A)
- net VDD_nRF: now also R4.1
- net at R14.2: now also U1.34 (AIN5/P0.29); no longer U1.4 (AIN2/P0.04)
- net at R13.2: now also U1.33 (AIN4/P0.28); no longer U1.36 (AIN7/P0.31)
- net at R15.2: now also U1.35 (AIN6/P0.30); no longer U1.5 (AIN3/P0.05)
- net MISO: no longer names the net of U1.32 (AIN0/P0.02)
- net MISO: no longer U2.1 (SDO/SA0)
- removed net MOSI: U1.33 (AIN4/P0.28), U2.14 (SDA)
- removed net SCK: U1.34 (AIN5/P0.29), U2.13 (SCL)
- no-connect marks 15 -> 19
Other:
- note removed: "near U3"
- moved on the sheet: D3, D4, D5, R1, R2, U3
