File: KICAD Projects/Primis_Locus/_restore_backup_2026-10-03T21-19-35-096/Locus.kicad_pcb (KiCad board)
At the start: 4 copper layers, 40 x 40 mm, 65 parts, among them J1 Conn_ARM_SWD_TagConnect_TC203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, J2 S2B-PH-SM4-TB_LF_SN, J4 USB_C_Receptacle_USB2.0_16P, SW1 SW_DPST_x2, U1 nRF52833_QDxx, U2 LSM6DSV16XTR, U3 LP5817DRLR, U5 MCP73831T-2ATI_OT, Y1 32.768kHz, Y2 32MHz

Commit message: ev2 wip1
Parts:
- added R4: 4.7k, Resistor_SMD:R_0402_1005Metric, F.Cu at (203.0, 49.8)
- moved TP4 15.6 mm to (208.0, 82.8)
- moved R2 7.77 mm to (199.5, 49.8)
- moved C13 7.66 mm to (204.5, 53.5), turned to 90 degrees
- moved R1 7.21 mm to (201.2, 49.8), turned to -90 degrees
- moved R13 6.75 mm to (203.2, 61.0)
- moved D2 5.45 mm to (201.3, 58.2), turned to 0 degrees
- moved U2 5.00 mm to (201.2, 53.2), turned to 0 degrees
- moved R15 4.79 mm to (198.5, 57.2), turned to 180 degrees
- moved C10 4.00 mm to (205.0, 59.8)
- moved TP2 3.61 mm to (194.5, 52.5)
- moved R14 3.03 mm to (198.5, 58.8)
- moved C29 2.61 mm to (201.3, 61.2), turned to 0 degrees
- moved TP1 2.29 mm to (191.4, 54.0)
- moved TP3 2.07 mm to (193.0, 79.0)
- moved C12 2.02 mm to (200.3, 56.0), turned to 0 degrees
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Connections:
- R13 pad 2: Net-(U1-AIN7/P0.31) -> Net-(U1-AIN4/P0.28)
- R14 pad 2: Net-(U1-AIN2/P0.04) -> Net-(U1-AIN5/P0.29)
- R15 pad 2: Net-(U1-AIN3/P0.05) -> Net-(U1-AIN6/P0.30)
- U1 pad 14: unconnected-(U1-P0.15-Pad14) -> INT
- U1 pad 31: INT -> unconnected-(U1-AIN1/P0.03-Pad31)
- U1 pad 32: MISO -> unconnected-(U1-AIN0/P0.02-Pad32)
- U1 pad 33: MOSI -> Net-(U1-AIN4/P0.28)
- U1 pad 34: SCK -> Net-(U1-AIN5/P0.29)
- U1 pad 35: CS -> Net-(U1-AIN6/P0.30)
- U1 pad 36: Net-(U1-AIN7/P0.31) -> unconnected-(U1-AIN7/P0.31-Pad36)
- U1 pad 4: Net-(U1-AIN2/P0.04) -> unconnected-(U1-AIN2/P0.04-Pad4)
- U1 pad 5: Net-(U1-AIN3/P0.05) -> unconnected-(U1-AIN3/P0.05-Pad5)
- U2 pad 1: MISO -> GND
- U2 pad 13: SCK -> SCL
- U2 pad 14: MOSI -> SDA
Routing:
- net SDA: track 21.1 -> 40.6 mm
- net INT: track 10.5 -> 29.9 mm, vias 0 -> 2
- net SCL: track 21.5 -> 39.7 mm
- net VDDH: track 111.7 -> 94.4 mm
- net Net-(U1-AIN3/P0.05): track 10.5 -> 0.00 mm, vias 2 -> 0
- net VDD_nRF: track 88.5 -> 98.7 mm
- net Net-(U1-AIN6/P0.30): track 0.00 -> 9.64 mm, vias 0 -> 2
- net Net-(U1-AIN2/P0.04): track 9.20 -> 0.00 mm, vias 2 -> 0
- net Net-(U1-AIN7/P0.31): track 8.95 -> 0.00 mm
- net Net-(U1-AIN5/P0.29): track 0.00 -> 8.36 mm, vias 0 -> 2
- net MISO: track 6.19 -> 0.00 mm
- net SCK: track 6.19 -> 0.00 mm
- net MOSI: track 6.14 -> 0.00 mm
- net DEC4_6: track 27.1 -> 22.4 mm
- net Net-(U1-AIN4/P0.28): track 0.00 -> 3.98 mm
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