File: KICAD Projects/Primis_Locus/_restore_backup_2026-10-04T00-52-15-244/Locus.kicad_sch (KiCad schematic)
At the start: 61 parts, among them J1 Conn_ARM_SWD_TagConnect_TC203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, J2 S2B-PH-SM4-TB_LF_SN, J4 USB_C_Receptacle_USB2.0_16P, SW1 SW_DPST_x2, U1 nRF52833_QDxx, U2 LSM6DSV16XTR, U3 LP5817DRLR, U5 MCP73831T-2ATI_OT, Y1 32.768kHz, Y2 32MHz

Commit message: ev2 wip1
Parts:
- added R4: 4.7k, Resistor_SMD:R_0402_1005Metric, symbol Device:R
Connections:
- net CS: now also R4.2; no longer U1.35 (AIN6/P0.30)
- net GND: no longer U2.2 (SDX/AH1/QVAR1), U2.3 (SCX/AH2/QVAR2)
- net INT: now also U1.14 (P0.15); no longer U1.31 (AIN1/P0.03)
- net MISO: no longer U1.32 (AIN0/P0.02)
- net MOSI: now also U2.2 (SDX/AH1/QVAR1); no longer U1.33 (AIN4/P0.28), U2.14 (SDA)
- net SCK: now also U2.3 (SCX/AH2/QVAR2); no longer U1.34 (AIN5/P0.29), U2.13 (SCL)
- net VDD_nRF: now also R4.1
- net at R14.2: now also U1.34 (AIN5/P0.29); no longer U1.4 (AIN2/P0.04)
- net at R13.2: now also U1.33 (AIN4/P0.28); no longer U1.36 (AIN7/P0.31)
- net at R15.2: now also U1.35 (AIN6/P0.30); no longer U1.5 (AIN3/P0.05)
- no-connect marks 15 -> 21
Other:
- note removed: "near U3"
- moved on the sheet: C15, D3, D4, D5, R1, R2, U3
