File: KICAD Projects/Primis_Locus/_restore_backup_2026-10-04T13-43-02-671/Locus.kicad_pcb (KiCad board)
At the start: 4 copper layers, 40 x 40 mm, 65 parts, among them J1 Conn_ARM_SWD_TagConnect_TC203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, J2 S2B-PH-SM4-TB_LF_SN, J4 USB_C_Receptacle_USB2.0_16P, SW1 SW_DPST_x2, U1 nRF52833_QDxx, U2 LSM6DSV16XTR, U3 LP5817DRLR, U5 MCP73831T-2ATI_OT, Y1 32.768kHz, Y2 32MHz

Commit message: ev2 wip1
Parts:
- moved R2 2.67 mm to (205.5, 52.4)
- moved R1 2.15 mm to (206.6, 52.5), turned to -90 degrees
- moved C1 0.67 mm to (196.8, 65.3)
- moved C10 0.54 mm to (205.0, 63.4)
- moved C8 0.30 mm to (202.5, 72.0)
Routing:
- net DEC4_6: track 27.1 -> 5.51 mm, vias 2 -> 0
- net SCL: track 21.5 -> 0.00 mm, vias 2 -> 0
- net SDA: track 21.1 -> 0.00 mm, vias 2 -> 0
- net VDD_nRF: track 88.5 -> 73.0 mm
- net GND: track 58.5 -> 56.0 mm, vias 99 -> 98
- net VDDH: track 111.7 -> 110.6 mm
- net Net-(U1-DEC1): track 1.57 -> 2.08 mm
