File: KICAD Projects/Primis_Locus/_restore_backup_2026-10-04T13-43-02-671/Locus.kicad_sch (KiCad schematic)
At the start: 61 parts, among them J1 Conn_ARM_SWD_TagConnect_TC203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, J2 S2B-PH-SM4-TB_LF_SN, J4 USB_C_Receptacle_USB2.0_16P, SW1 SW_DPST_x2, U1 nRF52833_QDxx, U2 LSM6DSV16XTR, U3 LP5817DRLR, U5 MCP73831T-2ATI_OT, Y1 32.768kHz, Y2 32MHz

Commit message: ev2 wip1
Connections:
- no-connect marks 15 -> 14
Changed lines of the file:
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@@
-	)
-	(no_connect
-		(at 128.27 120.65)
 	)
 	(no_connect
