File: KICAD Projects/Primis_Locus/Locus.kicad_sch (KiCad schematic)
At the start: 61 parts, among them J1 Conn_ARM_SWD_TagConnect_TC203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, J2 S2B-PH-SM4-TB_LF_SN, J4 USB_C_Receptacle_USB2.0_16P, SW1 SW_DPST_x2, U1 nRF52833_QDxx, U2 LSM6DSV16XTR, U3 LP5817DRLR, U5 MCP73831T-2ATI_OT, Y1 32.768kHz, Y2 32MHz

Commit message: ev2 pr
Changed lines of the file:
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@@
 		(in_pos_files yes)
 		(dnp no)
-		(fields_autoplaced yes)
 		(property "Reference" "R2"
-			(at 227.33 55.8799 0)
+			(at 226.568 55.88 0)
 			(show_name no)
 			(do_not_autoplace no)
@@
 		)
 		(property "Value" "4.7k"
-			(at 227.33 58.4199 0)
+			(at 226.314 58.42 0)
 			(show_name no)
 			(do_not_autoplace no)
