File: KICAD Projects/Primis_Locus/Locus.kicad_pcb (KiCad board)
At the start: 4 copper layers, 40 x 40 mm, 65 parts, among them J1 Conn_ARM_SWD_TagConnect_TC203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, J2 S2B-PH-SM4-TB_LF_SN, J4 USB_C_Receptacle_USB2.0_16P, SW1 SW_DPST_x2, U1 nRF52833_QDxx, U2 LSM6DSV16XTR, U3 LP5817DRLR, U5 MCP73831T-2ATI_OT, Y1 32.768kHz, Y2 32MHz

Commit message: ev2 pr
Parts:
- moved G*** 0.11 mm to (215.3, 78.7)
- moved R2 0.09 mm to (205.1, 55.1)
- moved R1 0.07 mm to (206.5, 54.6)
- moved D4 0.06 mm to (219.2, 49.6)
Routing:
- net VDD_nRF: track 88.5 -> 83.2 mm
- net VDDH: track 111.7 -> 110.0 mm
- net GND: track 58.5 -> 59.3 mm, vias 99 -> 98
